File: ELE_sch/kicad_proj/L1_RF_OPTICAL_tests_sch/ESP32_carrier_board.kicad_sch (KiCad schematic)
At the start: 2 parts, among them U7 433MHz_module_transmitter, U8 CC1101_MODULE

Commit message: schematics almost final (need confirmation of voltages of 433 mhz modules data pins)
Parts:
- added C16: 100uF, symbol Device:C_Polarized
- added C17, C18, C20: 4.7uF, symbol Device:C_Polarized
- added C19, C21: 100nF, symbol Device:C
- added C23, C26: 22uF/10V, symbol Device:C_Polarized
- added C24: 47uF, symbol Device:C_Polarized
- added C25: 120uF, symbol Device:C_Polarized
- added D2: LED, symbol Device:LED
- added J4, J5: 5V IN/OUT, symbol Connector_Generic:Conn_01x02
- added J6: OPTICAL TRANSMITTER SIGNAL from ESP32, symbol Connector_Generic:Conn_01x02
- added R6: 680R, symbol Device:R
- added R7: 10k, symbol Device:R
- added R8: 220R, symbol Device:R
- added U6: MCP1826S-33, symbol Regulator_Linear:MCP1826S
Connections:
- net at U7.1 (DATA): now also R8.2
- net +5V: now reaches U7.2 (VCC)
- net +5V: now also C16.1, C17.1, C18.1, C19.1, C25.1, C26.1, J4.1 (Pin_1), J5.1 (Pin_1), U6.1 (VI)
- net GND_ESP32: now reaches U7.3 (GND)
- net GND_ESP32: now also U8.1 (GND), C16.2, C17.2, C18.2, C19.2, C20.2, C21.2, C23.2, C24.2, C25.2, C26.2, J4.2 (Pin_2), J5.2 (Pin_2), J6.1 (Pin_1), U6.2 (GND)
- net +3V3_ESP32: now reaches U8.2 (VCC)
- net +3V3_ESP32: now also C20.1, C21.1, C23.1, C24.1, D2.2 (A), R7.2, U6.3 (VO)
- net ESP32_CC1101_GDO0(GPIO26): now reaches U8.3 (GDO0)
- net ESP32_CC1101_CSN(GPIO21): now reaches U8.4 (CSN)
- net ESP32_CC1101_CSN(GPIO21): now also R7.1
- net ESP32_VSPI_SCK(GPIO18): now reaches U8.5 (SCK)
- net ESP32_VSPI_MOSI(GPIO23): now reaches U8.6 (MOSI)
- net ESP32_VSPI_MISO(GPIO19): now reaches U8.7 (MISO)
- net ESP32_CC1101_GDO2(GPIO27): now reaches U8.8 (GDO2)
- new net: D2.1 (K), R6.1
- new net 433_ESP_DATA: R8.1
- new net ESP32_OPTIC_TX_EXT: J6.2 (Pin_2)
- no-connect marks 0 -> 10
Other:
- note added: "SIMPLIFIED ESP32-WROOM-32D DEVKIT BLOCK"
- title: RF transmission path circuits -> ESP32-WROOM-32D carrier with RF transmission path circuits
- moved on the sheet: U7, U8
