File: ELE_sch/kicad_proj/L1_RF_OPTICAL_tests_sch/STM32_carrier_board.kicad_sch (KiCad schematic)
At the start: 24 parts, among them J1 5V IN/OUT, J2 5V IN/OUT, J3 OPTICAL RECEIVER SIGNAL to ST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, U1 CC1101_MODULE, U2 AMS1117-3.3, U3 433MHz_module_receiver, U4 MH_Level_converter

Commit message: schematics almost final (need confirmation of voltages of 433 mhz modules data pins)
Connections:
- net STM32_SPI1_MISO(PA6): now also U1.7 (MISO); no longer U1.6 (MOSI)
- net STM32_SPI1_MOSI(PA7): now also U1.6 (MOSI); no longer U1.7 (MISO)
Other:
- title: RF transmission path circuits -> STM32H743 carrier with RF transmission path circuits
Changed lines of the file:
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@@
 	(paper "A3")
 	(title_block
-		(title "RF transmission path circuits")
+		(title "STM32H743 carrier with RF transmission path circuits")
 		(date "2026-10-25")
 		(rev "v1.0")
@@
 	(wire
 		(pts
-			(xy 215.138 218.186) (xy 237.744 218.186)
+			(xy 298.958 162.56) (xy 304.8 162.56)
 		)
 		(stroke
@@
 	(wire
 		(pts
-			(xy 298.704 162.56) (xy 304.8 162.56)
+			(xy 215.138 218.186) (xy 237.744 218.186)
 		)
 		(stroke
@@
 	(wire
 		(pts
+			(xy 298.958 161.544) (xy 298.958 162.56)
+		)
+		(stroke
+			(width 0)
+			(type default)
+		)
+	)
+	(wire
+		(pts
 			(xy 189.738 218.694) (xy 189.738 225.552)
 		)
@@
 	(wire
 		(pts
-			(xy 269.748 190.5) (xy 304.8 190.5)
+			(xy 270.002 190.5) (xy 304.8 190.5)
 		)
 		(stroke
@@
 		)
 	)
-	(label "STM32_SPI1_MISO(PA6)"
-		(at 241.808 177.8 180)
-		(effects
-			(font
-				(size 1.27 1.27)
-			)
-			(justify right bottom)
-		)
-	)
 	(label "STM32_COMP2_INM(PE7)"
 		(at 370.332 180.34 180)
@@
 		)
 	)
+	(label "STM32_SPI1_MOSI(PA7)"
+		(at 241.808 177.8 180)
+		(effects
+			(font
+				(size 1.27 1.27)
+			)
+			(justify right bottom)
+		)
+	)
 	(label "STM32_CC1101_GDO0(PB0)"
 		(at 162.052 177.8 0)
@@
 		)
 	)
-	(label "STM32_SPI1_MOSI(PA7)"
-		(at 241.808 175.26 180)
-		(effects
-			(font
-				(size 1.27 1.27)
-			)
-			(justify right bottom)
-		)
-	)
 	(label "STM32_COMP2_OUT(PE8)"
 		(at 370.332 175.26 180)
@@
 		)
 	)
+	(label "STM32_SPI1_MISO(PA6)"
+		(at 241.808 175.26 180)
+		(effects
+			(font
+				(size 1.27 1.27)
+			)
+			(justify right bottom)
+		)
+	)
 	(label "433_STM_DATA_HV"
 		(at 166.37 113.284 0)
@@
 	)
 	(label "STM32_CC1101_GDO0(PB0)"
-		(at 269.748 190.5 0)
+		(at 270.002 190.5 0)
 		(effects
 			(font
@@
 	)
 	(symbol
-		(lib_id "power:+3V3")
-		(at 298.704 162.56 0)
+		(lib_id "power:GND")
+		(at 67.056 159.512 0)
+		(mirror y)
 		(unit 1)
 		(body_style 1)
@@
 		(in_pos_files yes)
 		(dnp no)
-		(property "Reference" "#PWR030"
-			(at 298.704 166.37 0)
+		(property "Reference" "#PWR011"
+			(at 67.056 165.862 0)
 			(hide yes)
 			(show_name no)
@@
 			)
 		)
-		(property "Value" "+3V3_STM32"
-			(at 298.196 159.004 0)
+		(property "Value" "GND_STM32"
+			(at 66.04 154.686 90)
 			(show_name no)
 			(do_not_autoplace no)
@@
 		)
 		(property "Footprint" ""
-			(at 298.704 162.56 0)
+			(at 67.056 159.512 0)
 			(hide yes)
 			(show_name no)
@@
 		)
 		(property "Datasheet" ""
-			(at 298.704 162.56 0)
+			(at 67.056 159.512 0)
 			(hide yes)
 			(show_name no)
@@
 			)
 		)
-		(property "Description" "Power symbol creates a global label with name \"+3V3\""
-			(at 298.704 162.56 0)
+		(property "Description" "Power symbol creates a global label with name \"GND\" , ground"
+			(at 67.056 159.512 0)
 			(hide yes)
 			(show_name no)
@@
 			(project "L1_RF_OPTICAL_tests_sch"
 				(path "/8a635b1b-9d9a-4020-b936-45919ee57615/ccc22324-4fc6-46a7-86c7-31621d9abc7c"
-					(reference "#PWR030")
+					(reference "#PWR011")
 					(unit 1)
 				)
@@
 	)
 	(symbol
-		(lib_id "power:GND")
-		(at 67.056 159.512 0)
-		(mirror y)
+		(lib_id "power:+3V3")
+		(at 62.484 159.258 0)
+		(mirror x)
 		(unit 1)
 		(body_style 1)
@@
 		(in_pos_files yes)
 		(dnp no)
-		(property "Reference" "#PWR011"
-			(at 67.056 165.862 0)
+		(property "Reference" "#PWR012"
+			(at 62.484 155.448 0)
 			(hide yes)
 			(show_name no)
@@
 			)
 		)
-		(property "Value" "GND_STM32"
-			(at 66.04 154.686 90)
+		(property "Value" "+3V3_STM32"
+			(at 60.706 154.94 90)
 			(show_name no)
 			(do_not_autoplace no)
@@
 		)
 		(property "Footprint" ""
-			(at 67.056 159.512 0)
+			(at 62.484 159.258 0)
 			(hide yes)
 			(show_name no)
@@
 		)
 		(property "Datasheet" ""
-			(at 67.056 159.512 0)
+			(at 62.484 159.258 0)
 			(hide yes)
 			(show_name no)
@@
 			)
 		)
-		(property "Description" "Power symbol creates a global label with name \"GND\" , ground"
-			(at 67.056 159.512 0)
+		(property "Description" "Power symbol creates a global label with name \"+3V3\""
+			(at 62.484 159.258 0)
 			(hide yes)
 			(show_name no)
@@
 			(project "L1_RF_OPTICAL_tests_sch"
 				(path "/8a635b1b-9d9a-4020-b936-45919ee57615/ccc22324-4fc6-46a7-86c7-31621d9abc7c"
-					(reference "#PWR011")
+					(reference "#PWR012")
 					(unit 1)
 				)
@@
 	)
 	(symbol
-		(lib_id "power:+3V3")
-		(at 62.484 159.258 0)
-		(mirror x)
+		(lib_id "power:GND")
+		(at 234.188 67.31 0)
 		(unit 1)
 		(body_style 1)
@@
 		(in_pos_files yes)
 		(dnp no)
-		(property "Reference" "#PWR012"
-			(at 62.484 155.448 0)
+		(property "Reference" "#PWR021"
+			(at 234.188 73.66 0)
 			(hide yes)
 			(show_name no)
@@
 			)
 		)
-		(property "Value" "+3V3_STM32"
-			(at 60.706 154.94 90)
+		(property "Value" "GND_STM32"
+			(at 234.188 71.12 0)
 			(show_name no)
 			(do_not_autoplace no)
@@
 		)
 		(property "Footprint" ""
-			(at 62.484 159.258 0)
+			(at 234.188 67.31 0)
 			(hide yes)
 			(show_name no)
@@
 		)
 		(property "Datasheet" ""
-			(at 62.484 159.258 0)
+			(at 234.188 67.31 0)
 			(hide yes)
 			(show_name no)
@@
 			)
 		)
-		(property "Description" "Power symbol creates a global label with name \"+3V3\""
-			(at 62.484 159.258 0)
+		(property "Description" "Power symbol creates a global label with name \"GND\" , ground"
+			(at 234.188 67.31 0)
 			(hide yes)
 			(show_name no)
@@
 			(project "L1_RF_OPTICAL_tests_sch"
 				(path "/8a635b1b-9d9a-4020-b936-45919ee57615/ccc22324-4fc6-46a7-86c7-31621d9abc7c"
-					(reference "#PWR012")
+					(reference "#PWR021")
 					(unit 1)
 				)
@@
 	)
 	(symbol
-		(lib_id "power:GND")
-		(at 234.188 67.31 0)
+		(lib_id "power:+5V")
+		(at 298.958 161.544 0)
 		(unit 1)
 		(body_style 1)
@@
 		(in_pos_files yes)
 		(dnp no)
-		(property "Reference" "#PWR021"
-			(at 234.188 73.66 0)
+		(property "Reference" "#PWR030"
+			(at 298.958 165.354 0)
 			(hide yes)
 			(show_name no)
@@
 			)
 		)
-		(property "Value" "GND_STM32"
-			(at 234.188 71.12 0)
+		(property "Value" "+5V"
+			(at 298.958 157.734 0)
 			(show_name no)
 			(do_not_autoplace no)
@@
 		)
 		(property "Footprint" ""
-			(at 234.188 67.31 0)
+			(at 298.958 161.544 0)
 			(hide yes)
 			(show_name no)
@@
 		)
 		(property "Datasheet" ""
-			(at 234.188 67.31 0)
+			(at 298.958 161.544 0)
 			(hide yes)
 			(show_name no)
@@
 			)
 		)
-		(property "Description" "Power symbol creates a global label with name \"GND\" , ground"
-			(at 234.188 67.31 0)
+		(property "Description" "Power symbol creates a global label with name \"+5V\""
+			(at 298.958 161.544 0)
 			(hide yes)
 			(show_name no)
@@
 			(project "L1_RF_OPTICAL_tests_sch"
 				(path "/8a635b1b-9d9a-4020-b936-45919ee57615/ccc22324-4fc6-46a7-86c7-31621d9abc7c"
-					(reference "#PWR021")
+					(reference "#PWR030")
 					(unit 1)
 				)
