File: ELE_sch/kicad_proj/L1_RF_OPTICAL_tests_sch/STM32_carrier_board.kicad_sch (KiCad schematic)
At the start: 24 parts, among them J1 5V IN/OUT, J2 5V IN/OUT, J3 OPTICAL RECEIVER SIGNAL to ST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, U1 CC1101_MODULE, U2 AMS1117-3.3, U3 433MHz_module_receiver, U4 MH_Level_converter

Commit message: set 433mhz receiver resistor according to measurements from osciloscope
Parts:
- added R9: 470R, symbol Device:R
Connections:
- net 433_STM_DATA_HV: now also R9.2; no longer U3.2 (DATA), U3.3 (DATA)
- new net: R9.1, U3.2 (DATA), U3.3 (DATA)
Changed lines of the file:
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@@
 	)
 	(junction
-		(at 188.214 118.618)
-		(diameter 0)
-		(color 0 0 0 0)
-	)
-	(junction
 		(at 176.784 116.078)
 		(diameter 0)
@@
 	)
 	(junction
+		(at 188.214 118.618)
+		(diameter 0)
+		(color 0 0 0 0)
+	)
+	(junction
 		(at 176.784 123.698)
 		(diameter 0)
@@
 	(wire
 		(pts
+			(xy 184.15 108.204) (xy 184.15 118.618)
+		)
+		(stroke
+			(width 0)
+			(type default)
+		)
+	)
+	(wire
+		(pts
 			(xy 270.002 170.18) (xy 304.8 170.18)
 		)
@@
 	(wire
 		(pts
+			(xy 184.15 118.618) (xy 188.214 118.618)
+		)
+		(stroke
+			(width 0)
+			(type default)
+		)
+	)
+	(wire
+		(pts
 			(xy 229.362 235.712) (xy 225.552 235.712)
 		)
@@
 	(wire
 		(pts
-			(xy 184.658 118.618) (xy 184.658 113.284)
+			(xy 183.642 108.204) (xy 184.15 108.204)
 		)
 		(stroke
@@
 	(wire
 		(pts
-			(xy 166.37 113.284) (xy 184.658 113.284)
+			(xy 156.718 108.204) (xy 176.022 108.204)
 		)
 		(stroke
@@
 	(wire
 		(pts
-			(xy 184.658 118.618) (xy 188.214 118.618)
-		)
-		(stroke
-			(width 0)
-			(type default)
-		)
-	)
-	(wire
-		(pts
 			(xy 187.706 180.34) (xy 162.052 180.34)
 		)
@@
 	)
 	(label "433_STM_DATA_HV"
-		(at 166.37 113.284 0)
+		(at 156.718 108.204 0)
 		(effects
 			(font
@@
 					(unit 1)
 				)
+			)
+		)
+	)
+	(symbol
+		(lib_id "Device:R")
+		(at 179.832 108.204 270)
+		(unit 1)
+		(body_style 1)
+		(exclude_from_sim no)
+		(in_bom yes)
+		(on_board yes)
+		(in_pos_files yes)
+		(dnp no)
+		(property "Reference" "R9"
+			(at 180.848 105.918 90)
+			(show_name no)
+			(do_not_autoplace no)
+			(effects
+				(font
+					(size 1.27 1.27)
+				)
+				(justify right)
+			)
+		)
+		(property "Value" "470R"
+			(at 181.102 110.744 90)
+			(show_name no)
+			(do_not_autoplace no)
+			(effects
+				(font
+					(size 1.27 1.27)
+				)
+				(justify right)
+			)
+		)
+		(property "Footprint" ""
+			(at 179.832 106.426 90)
+			(hide yes)
+			(show_name no)
+			(do_not_autoplace no)
+			(effects
+				(font
+					(size 1.27 1.27)
+				)
+			)
+		)
+		(property "Datasheet" ""
+			(at 179.832 108.204 0)
+			(hide yes)
+			(show_name no)
+			(do_not_autoplace no)
+			(effects
+				(font
+					(size 1.27 1.27)
+				)
+			)
+		)
+		(property "Description" "Resistor"
+			(at 179.832 108.204 0)
+			(hide yes)
+			(show_name no)
+			(do_not_autoplace no)
+			(effects
+				(font
+					(size 1.27 1.27)
+				)
+			)
+		)
+		(pin "2"
+		)
+		(pin "1"
+		)
+		(instances
+			(project "L1_RF_OPTICAL_tests_sch"
+				(path "/8a635b1b-9d9a-4020-b936-45919ee57615/ccc22324-4fc6-46a7-86c7-31621d9abc7c"
+					(reference "R9")
+					(unit 1)
+				)
