File: ELE_sch/kicad_proj/L1_RF_OPTICAL_tests_sch/optical_path.kicad_sch (KiCad schematic)
At the start: 5 parts

Commit message: schematics almost final (need confirmation of voltages of 433 mhz modules data pins)
Connections:
- net ESP32_GPIO renamed ESP32_OPTIC_TX_EXT
Changed lines of the file:
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@@
+	(wire
+		(pts
+			(xy 112.014 83.058) (xy 133.35 83.058)
+		)
+		(stroke
+			(width 0)
+			(type default)
+		)
+	)
 	(wire
 		(pts
@@
 	(wire
 		(pts
-			(xy 129.032 69.596) (xy 129.032 76.454)
+			(xy 129.032 69.596) (xy 129.032 75.946)
 		)
 		(stroke
@@
 	(wire
 		(pts
-			(xy 129.032 76.454) (xy 115.316 76.454)
+			(xy 129.032 75.946) (xy 108.966 75.946)
 		)
 		(stroke
@@
 		)
 	)
-	(label "ESP32_GPIO"
-		(at 115.316 76.454 0)
+	(label "TO_ESP32_OPTIC_TX"
+		(at 112.014 83.058 0)
+		(effects
+			(font
+				(size 1.27 1.27)
+			)
+			(justify left bottom)
+		)
+	)
+	(label "TO_ESP32_OPTIC_TX"
+		(at 108.966 75.946 0)
 		(effects
 			(font
@@
 		)
 	)
+	(global_label "ESP32_OPTIC_TX_EXT"
+		(shape input)
+		(at 133.35 83.058 0)
+		(fields_autoplaced yes)
+		(effects
+			(font
+				(size 1.27 1.27)
+			)
+			(justify left)
+		)
+		(property "Intersheetrefs" "${INTERSHEET_REFS}"
+			(at 156.2316 83.058 0)
+			(hide yes)
+			(show_name no)
+			(do_not_autoplace no)
+			(effects
+				(font
+					(size 1.27 1.27)
+				)
+				(justify left)
+			)
+		)
+	)
